File: tests/fixtures/DCCF.sved_placed.kicad_pcb (KiCad board)
At the start: 2 copper layers, 230.8 x 200 mm, 97 parts, among them J1 AudioJack2_SwitchT, J2 AudioJack2_SwitchT, J3 AudioJack2_SwitchT, J4 AudioJack2_SwitchT, J5 AudioJack2_SwitchT, J6 AudioJack2_SwitchT, Q1 Conn_01x07_Male, Q2 USB_B_Micro, SW1 SW_SPDT, SW2 SW_SPDT, SW3 SW_SPDT, SW4 SW_SPDT, SW5 SW_SPDT, SW6 SW_SPDT, T1 B1K, T2 B1K, U1 LM358, U2 LM324, U3 LM324, U4 LM324

Commit message: Per-region placement, routing infra, DRC + track rip-up, UI overhaul
- placement.py: per-region force simulation + shapely courtyard collision
- routing/: grid, obstacles, A* router, scheduler, output, pipeline
- drc.py: DRC runner; io.rip_up_nets + board_model.commit_placement
- ui: footprint sidebar, selection, forces overlay, layer/DRC toggles
- pyproject.toml editable install; shapely dep; start_server browser-open
- fix accept_proposal: unpack 3-tuple + set union for power nets
- track tube111 fixtures; gitignore tmp/
Parts:
- moved H9 171.0 mm to (184.5, 142.1)
- moved H3 142.7 mm to (187.2, 49.4)
- moved H15 138.6 mm to (183.1, 233.6)
- moved H8 135.1 mm to (135.6, 141.3)
- moved T1 130.9 mm to (244.9, 65.3), turned to 210.374 degrees
- moved SW5 129.9 mm to (263.6, 169.8), turned to 89.8344 degrees
- moved R5 121.5 mm to (250.9, 61.7), turned to 157.069 degrees
- moved T2 118.8 mm to (209.6, 63.2), turned to -33.2785 degrees
- moved J1 115.7 mm to (202.3, 64.1), turned to 15.5431 degrees
- moved C12 110.9 mm to (246.4, 210.5), turned to 92.4463 degrees
- moved J6 110.7 mm to (203.4, 204.6), turned to 14.123 degrees
- moved J5 106.6 mm to (203.1, 183.0), turned to 18.6306 degrees
- moved R4 106.6 mm to (246.6, 64.2), turned to -176.233 degrees
- moved RV2 106.4 mm to (264.1, 90.2), turned to 150.05 degrees
- moved H10 100.6 mm to (268.7, 141.7)
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