File: tests/fixtures/DCCF.2a-modified.kicad_pcb (KiCad board)
At the start: 2 copper layers, 230.8 x 200 mm, 97 parts, among them J1 AudioJack2_SwitchT, J2 AudioJack2_SwitchT, J3 AudioJack2_SwitchT, J4 AudioJack2_SwitchT, J5 AudioJack2_SwitchT, J6 AudioJack2_SwitchT, Q1 Conn_01x07_Male, Q2 USB_B_Micro, SW1 SW_SPDT, SW2 SW_SPDT, SW3 SW_SPDT, SW4 SW_SPDT, SW5 SW_SPDT, SW6 SW_SPDT, T1 B1K, T2 B1K, U1 LM358, U2 LM324, U3 LM324, U4 LM324

Commit message: Full-scale benchmark retest, measured perf fixes, docs pipeline repair
Benchmarks: new scripts/benchmark_stitch_pour.py (pour + stitch cost, budget sweep); all five benchmarks rerun full-scale with results in docs/benchmarks/. Fixed benchmark_routing --with-stitch fixture-name crash. Perf (measured, parity-verified): placement is_empty per-footprint cache (DCCF 55.7->19.4 ms/iter); pour disc painting via numba stamp_discs (tube111 pour 4.78->1.82s). GUI pre-flight estimates recalibrated (placement coefficient, routing seconds + stitch surcharge). In-tree SI work included: wall_exponent program (norm docs, params plumb-through, tight tests, DCCF fixture). Docs: Quarto book renders again (dangling filter removed, freeze:auto, portable pytest cells, pytest-html dev dep); primer boundary section + exponent docs; PLAN R8 status audit; TODO/VIN-bug/zone/weight notes in docs/benchmark_notes_2026-10-15.md.
Parts:
- moved R5 4.79 mm to (264.0, 61.7), turned to -145.141 degrees
- turned U2 to 88.603 degrees
